Commit message: URDF 중간저장 부피
파일 중간 저장

File: ROS/3.URDF/bumperbot.urdf (robot description, URDF)
Before this commit: robot bumperbot, 6 links, 5 joints
Links:
- link base_link: geometry collision mesh filename=package://bumperbot_description/meshes/base_link.STL; visual mesh filename=package://bumperbot_description/meshes/base_link.STL
