Commit message: 불필요한 내용 수정

File: ROS Project/ROS2/Project/1. Robot Arm/4) rviz/urdf/arms.urdf (robot description, URDF)
Before this commit: robot arms, 5 links, 5 joints
Links:
- added link link_4, mass 0.01; collision cylinder length=0.1 radius=0.06; visual cylinder length=0.1 radius=0.06
- added link link_5, mass 0.01; collision cylinder length=0.3 radius=0.03; visual cylinder length=0.3 radius=0.03
- link base_link: mass None -> 5.0
- link link_1: mass None -> 5.0
- link link_2: mass None -> 2.0
- link link_3: mass None -> 0.01
Joints:
- removed joint joint_base
- added joint joint_4: type continuous, parent link_3, child link_4, origin xyz= 0 0 -0.25 rpy=1.57 0 0, axis  0 0 1, limit lower=-1.92 upper=1.92 effort=10 velocity=0.5
- added joint joint_5: type fixed, parent link_4, child link_5, origin xyz=0.0 -0.2 0  rpy=1.57 0 0
- joint joint_2: limit (none) -> lower=-0.25 upper=3.34 effort=10 velocity=0.5
